Commit message: updated files

File: body.urdf (robot description, URDF)
Before this commit: robot robot, 9 links, 8 joints
Links:
- added link LeftLeftLeg, mass 1; collision box size=1 0.2 0.2; visual box size=1 0.2 0.2
- added link LeftLeftLowerLeg, mass 1; collision box size=0.2 0.2 1; visual box size=0.2 0.2 1
- added link RightRightLeg, mass 1; collision box size=1 0.2 0.2; visual box size=1 0.2 0.2
- added link RightRightLowerLeg, mass 1; collision box size=0.2 0.2 1; visual box size=0.2 0.2 1
Joints:
- added joint LeftLeftLeg_LowerLeftLeftLeg: type revolute, parent LeftLeftLeg, child LeftLeftLowerLeg, origin xyz=-1 0 0 rpy=0 0 0, axis 0 1 0, limit lower=-3.14159 upper=3.14159 effort=0.0 velocity=0.0
- added joint RightRightLeg_LowerRightRightLeg: type revolute, parent RightRightLeg, child RightRightLowerLeg, origin xyz=1 0 0 rpy=0 0 0, axis 0 1 0, limit lower=-3.14159 upper=3.14159 effort=0.0 velocity=0.0
- added joint Torso_LeftLeftLeg: type revolute, parent Torso, child LeftLeftLeg, origin xyz=-0.5 0.3 1 rpy=0 0 0, axis 0 1 0, limit lower=-3.14159 upper=3.14159 effort=0.0 velocity=0.0
- added joint Torso_RightRightLeg: type revolute, parent Torso, child RightRightLeg, origin xyz=0.5 -0.3 1 rpy=0 0 0, axis 0 1 0, limit lower=-3.14159 upper=3.14159 effort=0.0 velocity=0.0
- joint Torso_LeftLeg: origin xyz=-0.5 0 1 rpy=0 0 0 -> xyz=-0.5 -0.3 1 rpy=0 0 0
- joint Torso_RightLeg: origin xyz=0.5 0 1 rpy=0 0 0 -> xyz=0.5 0.3 1 rpy=0 0 0

Commit message: updated files

File: body.urdf (robot description, URDF)
Before this commit: robot robot, 13 links, 12 joints
Links:
- removed link LeftLeftLeg
- removed link LeftLeftLowerLeg
- removed link RightRightLeg
- removed link RightRightLowerLeg
Joints:
- removed joint LeftLeftLeg_LowerLeftLeftLeg
- removed joint RightRightLeg_LowerRightRightLeg
- removed joint Torso_LeftLeftLeg
- removed joint Torso_RightRightLeg
- joint Torso_LeftLeg: origin xyz=-0.5 -0.3 1 rpy=0 0 0 -> xyz=-0.5 0 1 rpy=0 0 0
- joint Torso_RightLeg: origin xyz=0.5 0.3 1 rpy=0 0 0 -> xyz=0.5 0 1 rpy=0 0 0

Commit message: updated files

File: body.urdf (robot description, URDF)
Before this commit: robot robot, 13 links, 12 joints
Joints:
- removed joint LeftLeftLeg_LowerLeftLeftLeg
- removed joint RightRightLeg_LowerRightRightLeg
- added joint LeftLeftLeg_LeftLeftLowerLeg: type revolute, parent LeftLeftLeg, child LeftLeftLowerLeg, origin xyz=-1 0 0 rpy=0 0 0, axis 0 1 0, limit lower=-3.14159 upper=3.14159 effort=0.0 velocity=0.0
- added joint RightRightLeg_RightRightLowerLeg: type revolute, parent RightRightLeg, child RightRightLowerLeg, origin xyz=1 0 0 rpy=0 0 0, axis 0 1 0, limit lower=-3.14159 upper=3.14159 effort=0.0 velocity=0.0
